Commit message: Added suuport for leader arm

File: soarm101_bringup/urdf/full.xacro (robot description, xacro)
@@ -2,7 +2,13 @@
 <robot xmlns:xacro="http://www.ros.org/wiki/xacro" name="soarm101">
   <!-- Аргумент выбора режима (sim / real) -->
-  <xacro:arg name="use_sim" default="true"/>
+  <xacro:arg name="use_sim" default="false"/>
+  <xacro:arg name="arm_type" default="follower"/>
+  <xacro:arg name="port" default="/dev/ttyACM0"/>
+  <xacro:arg name="max_speed" default="2400"/>
+  <xacro:arg name="max_accel" default="50"/>
+  <xacro:property name="arm_type" value="$(arg arm_type)" />
   <!-- URDF_description of SOARM101 -->
   <xacro:include filename="$(find soarm101_description)/urdf/soarm101.xacro"/>
+  <xacro:include filename="$(find soarm101_ros2_control)/urdf/ros2_control_real.xacro"/>
   <!--=================== ROS2_CONTROL & PLUGINS ===================-->
   <!-- Выбор варианта в зависимости от аргумента use_sim -->
@@ -13,5 +19,10 @@
   <xacro:unless value="$(arg use_sim)">
     <!-- РЕАЛЬНЫЙ РОБОТ -->
-    <xacro:include filename="$(find soarm101_ros2_control)/urdf/ros2_control_real.xacro"/>
+    <xacro:if value="${arm_type == 'leader'}">
+      <xacro:soarm101_hardware_leader port="$(arg port)" max_speed="$(arg max_speed)" max_accel="$(arg max_accel)"/>
+    </xacro:if>
+    <xacro:if value="${arm_type == 'follower'}">
+      <xacro:soarm101_hardware_follower port="$(arg port)" max_speed="$(arg max_speed)" max_accel="$(arg max_accel)"/>
+    </xacro:if>
   </xacro:unless>
 </robot>

File: soarm101_ros2_control/urdf/ros2_control_real.xacro (robot description, xacro)
@@ -1,18 +1,6 @@
 <?xml version="1.0"?>
 <robot xmlns:xacro="http://www.ros.org/wiki/xacro">
-  <ros2_control name="RealRobotSystem" type="system">
-    <hardware>
-      <plugin>soarm101_hardware/SOARM101SystemHardware</plugin>
-      <!-- Параметры, передаваемые в ваш плагин -->
-      <param name="port">/dev/ttyACM0</param>
-      <param name="baudrate">1000000</param>
-      <param name="default_speed">2400</param>
-      <param name="default_accel">50</param>
-      <param name="park_positions">[0.004, -1.712, 1.560, 1.141, -0.029, 0.461]</param>
-      <param name="calibration_file">$(find converter_calibration_data)/config/motor_calibration.yaml</param>
-      <!-- другие параметры -->
-    </hardware>
-    <!-- Интерфейсы для каждого сустава -->
-    <joint name="shoulder_pan_joint">
+  <xacro:macro name="joint_servo_with_command" params="joint_name">
+    <joint name="${joint_name}">
       <command_interface name="position"/>
       <state_interface name="position"/>
@@ -24,6 +12,7 @@
       <state_interface name="moving_flag"/>
     </joint>
-    <joint name="shoulder_lift_joint">
-      <command_interface name="position"/>
+  </xacro:macro>
+  <xacro:macro name="joint_servo_without_command" params="joint_name">
+    <joint name="${joint_name}">
       <state_interface name="position"/>
       <state_interface name="velocity"/>
@@ -34,44 +23,48 @@
       <state_interface name="moving_flag"/>
     </joint>
-    <joint name="elbow_flex_joint">
-      <command_interface name="position"/>
-      <state_interface name="position"/>
-      <state_interface name="velocity"/>
-      <state_interface name="effort"/>
-      <state_interface name="temperature"/>
-      <state_interface name="voltage"/>
-      <state_interface name="current"/>
-      <state_interface name="moving_flag"/>
-    </joint>
-    <joint name="wrist_flex_joint">
-      <command_interface name="position"/>
-      <state_interface name="position"/>
-      <state_interface name="velocity"/>
-      <state_interface name="effort"/>
-      <state_interface name="temperature"/>
-      <state_interface name="voltage"/>
-      <state_interface name="current"/>
-      <state_interface name="moving_flag"/>
-    </joint>
-    <joint name="wrist_roll_joint">
-      <command_interface name="position"/>
-      <state_interface name="position"/>
-      <state_interface name="velocity"/>
-      <state_interface name="effort"/>
-      <state_interface name="temperature"/>
-      <state_interface name="voltage"/>
-      <state_interface name="current"/>
-      <state_interface name="moving_flag"/>
-    </joint>
-    <joint name="gripper_jaw_joint">
-      <command_interface name="position"/>
-      <state_interface name="position"/>
-      <state_interface name="velocity"/>
-      <state_interface name="effort"/>
-      <state_interface name="temperature"/>
-      <state_interface name="voltage"/>
-      <state_interface name="current"/>
-      <state_interface name="moving_flag"/>
-    </joint>
-  </ros2_control>
+  </xacro:macro>
+  <xacro:macro name="soarm101_hardware_leader" params="port max_speed max_accel">
+    <ros2_control name="RealRobotSystem" type="system">
+      <hardware>
+        <plugin>soarm101_hardware/SOARM101SystemHardwareLeader</plugin>
+        <!-- params for plugin -->
+        <param name="port">${port}</param>
+        <param name="baudrate">1000000</param>
+        <param name="default_speed">${max_speed}</param>
+        <param name="default_accel">${max_accel}</param>
+        <param name="park_positions">[0.004, -1.712, 1.560, 1.141, -0.029, 0.461]</param>
+        <param name="max_torques">[2.69, 1.91, 2.69, 1.41, 1.41, 1.41]</param>
+        <param name="calibration_file">$(find converter_calibration_data)/config/leader_motor_calibration.yaml</param>
+      </hardware>
+      <!-- Interfaces for each joint -->
+      <xacro:joint_servo_without_command joint_name="shoulder_pan_joint" />
+      <xacro:joint_servo_without_command joint_name="shoulder_lift_joint" />
+      <xacro:joint_servo_without_command joint_name="elbow_flex_joint" />
+      <xacro:joint_servo_without_command joint_name="wrist_flex_joint" />
+      <xacro:joint_servo_without_command joint_name="wrist_roll_joint" />
+      <xacro:joint_servo_without_command joint_name="gripper_jaw_joint" />
+    </ros2_control>
+  </xacro:macro>
+  <xacro:macro name="soarm101_hardware_follower" params="port max_speed max_accel">
+    <ros2_control name="RealRobotSystem" type="system">
+      <hardware>
+        <plugin>soarm101_hardware/SOARM101SystemHardwareFollower</plugin>
+        <!-- params for plugin -->
+        <param name="port">${port}</param>
+        <param name="baudrate">1000000</param>
+        <param name="default_speed">${max_speed}</param>
+        <param name="default_accel">${max_accel}</param>
+        <param name="park_positions">[0.004, -1.712, 1.560, 1.141, -0.029, 0.461]</param>
+        <param name="max_torques">[2.94, 2.94, 2.94, 2.94, 2.94, 2.94]</param>
+        <param name="calibration_file">$(find converter_calibration_data)/config/follower_motor_calibration.yaml</param>
+      </hardware>
+      <!-- Interfaces for each joint -->
+      <xacro:joint_servo_with_command joint_name="shoulder_pan_joint" />
+      <xacro:joint_servo_with_command joint_name="shoulder_lift_joint" />
+      <xacro:joint_servo_with_command joint_name="elbow_flex_joint" />
+      <xacro:joint_servo_with_command joint_name="wrist_flex_joint" />
+      <xacro:joint_servo_with_command joint_name="wrist_roll_joint" />
+      <xacro:joint_servo_with_command joint_name="gripper_jaw_joint" />
+    </ros2_control>
+  </xacro:macro>
 </robot>

File: soarm101_ros2_control/urdf/ros2_control_sim.xacro (robot description, xacro)
@@ -1,5 +1,5 @@
 <?xml version="1.0"?>
 <robot xmlns:xacro="http://www.ros.org/wiki/xacro">
-  <!-- Плагин для Ignition Gazebo (gz_ros2_control) -->
+  <!-- Plugin for Ignition Gazebo (gz_ros2_control) -->
   <gazebo>
     <plugin filename="gz_ros2_control-system" name="gz_ros2_control::GazeboSimROS2ControlPlugin">
@@ -12,5 +12,5 @@
       <plugin>gz_ros2_control/GazeboSimSystem</plugin>
     </hardware>
-    <!-- Joints (имена остаются те же) -->
+    <!-- Joints  -->
     <joint name="shoulder_pan_joint">
       <command_interface name="position"/>
