Commit message: Devide URDF into several files and create urdf-agregator

File: soarm101_description/urdf/soarm101.xacro (robot description, xacro)
@@ -337,13 +337,3 @@
     <limit effort="10" velocity="10" lower="-1.91986" upper="1.91986"/>
   </joint>
-  <!--=================== ROS2_CONTROL & PLUGINS ===================-->
-  <!-- Выбор варианта в зависимости от аргумента use_sim -->
-  <xacro:if value="$(arg use_sim)">
-    <!-- СИМУЛЯЦИЯ -->
-    <xacro:include filename="$(find soarm101_ros2_control)/urdf/ros2_control_sim.xacro"/>
-  </xacro:if>
-  <xacro:unless value="$(arg use_sim)">
-    <!-- РЕАЛЬНЫЙ РОБОТ -->
-    <xacro:include filename="package://soarm101_description/urdf/ros2_control_real.xacro"/>
-  </xacro:unless>
 </robot>

File: soarm101_ros2_control/urdf/ros2_control_real.xacro (robot description, xacro)
@@ -5,5 +5,5 @@
       <plugin>soarm101_hardware/SOARM101Hardware</plugin>
       <!-- Параметры, передаваемые в ваш плагин -->
-      <param name="port">/dev/ttyUSB0</param>
+      <param name="port">/dev/ttyACM0</param>
       <param name="baudrate">1000000</param>
       <!-- другие параметры -->
@@ -35,5 +35,5 @@
       <state_interface name="velocity"/>
     </joint>
-    <joint name="gripper_joint">
+    <joint name="gripper_jaw_joint">
       <command_interface name="position"/>
       <state_interface name="position"/>

File: soarm101_ros2_control/urdf/ros2_control_sim.xacro (robot description, xacro)
@@ -4,5 +4,5 @@
   <gazebo>
     <plugin filename="gz_ros2_control-system" name="gz_ros2_control::GazeboSimROS2ControlPlugin">
-      <parameters>$(find soarm101_ros2_control)/config/sim_controllers.yaml</parameters>
+      <parameters>filename="package://soarm101_ros2_control/config/sim_controllers.yaml"</parameters>
     </plugin>
   </gazebo>

Commit message: Added new features for simultaneous work of both arms and teleoperation

File: soarm101_description/urdf/soarm101.xacro (robot description, xacro)
@@ -12,5 +12,5 @@
   </material>
   <!--=================== LINKS ===================-->
-  <link name="world"/>
+  <link name="zero_point_link"/>
   <!-- Link base -->
   <link name="base_link">
@@ -291,6 +291,6 @@
   </link>
   <!--=================== JOINTS ===================-->
-  <joint name="world_to_base_joint" type="fixed">
-    <parent link="world"/>
+  <joint name="zero_point_to_base_joint" type="fixed">
+    <parent link="zero_point_link"/>
     <child link="base_link"/>
     <origin xyz="-0.021 0.0485 -0.03" quat="0.0 0.0 -0.707108 0.707108"/>
